File: baseplate_test.kicad_sch (KiCad schematic)
At the start: 118 parts

Commit message: schematic finished (pretty much)
Parts:
- removed C? (x2): 0.1uF, 2_Passives_Capacitors_SMD_IPC:C_2012_805_B, symbol 2.passive:C
- removed C? (x2): 150uF, project_footprints:EMZR100ARA151ME61G, symbol 2.passive:CP1
- removed J?: LSHM-120-02.5-L-DV-A-S-K-TR, project_footprints:V_LSHM-120-02.5-L-DV-A-S-K-TR, symbol USB5537B:LSHM-120-02.5-L-DV-A-S-K-TR
- removed J?: header_01x04, 5_Connectors_misc:header_01x04_pitch2.54_tht, symbol 5.connector.interconnect:header_01x04
- removed U? (x2): Mounting-holes, 0_misc:plated_hole_2.2x3mm, symbol 5.connector.interconnect:Mounting-holes
- added C1: 1.0nF, 2_Passives_Capacitors_SMD_IPC:C_2012_805_B, symbol 2.passive:C
- added C14, C19: 0.1uF, 2_Passives_Capacitors_SMD_IPC:C_2012_805_B, symbol 2.passive:C
- added C42, C43, C44, C45, C46, C47, C48: 150uF, project_footprints:EMZR100ARA151ME61G, symbol 2.passive:CP1
- added C49, C50: 22uF, 2_Passives_Capacitors_SMD_IPC:C_2012_805_B, symbol 2.passive:C
- added C51: 47uF, 2_Passives_Capacitors_SMD_IPC:C_2012_805_B, symbol 2.passive:C
- added D10, D11, D9: GRN, 1_Semi_Discrete_Diodes_SMD:D_0805, symbol 1.semi.opto:LED
- added D8: D_Schottky, project_footprints:MBR1560STR, symbol 1.semi.discrete:D_Schottky
- added J1, J4, J5, J7, J8: USB3_A, project_footprints:USB3_A_Molex_48393-001, symbol 5.connector.interconnect.usb_dvi_hdmi:USB3_A
- added J10, J9: header_01x04, 5_Connectors_misc:header_01x04_pitch2.54_tht, symbol 5.connector.interconnect:header_01x04
- added J11, J12: header_01x05, 5_Connectors_misc:header_01x04_pitch2.54_tht, symbol 5.connector.interconnect:header_01x05
- added J2, J3, J6: USB_A, project_footprints:USB_A_Molex_67643_Horizontal, symbol 5.connector.interconnect.usb_dvi_hdmi:USB_A
- added R42: 267, project_footprints:RN55E2670BRE6, symbol 2.passive:R
- added R43: 140, 2_Passives_Resistors_SMD_IPC:R_2012_805_B, symbol 2.passive:R
- added R44, R45: 1.2k, 2_Passives_Resistors_SMD_IPC:R_6332_2512_B, symbol 2.passive:R
- added R46, R47: 110, 2_Passives_Resistors_SMD_IPC:R_2012_805_B, symbol 2.passive:R
- added TP6, TP7, TP8: TEST, 5_Connectors_misc:2mm_smd_pad, symbol 5.connector.interconnect:TEST
- added U9: OKR-T/10-W12, project_footprints:OKR-T_10-W12, symbol USB5537B:OKR-T/10-W12
- gave numbers to parts that had none: 110
Connections:
- net +3.3V: now also J10.2, J11.4, J12.4, TP8.1
- net +3V3: now also D11.1 (K), J11.3, J12.3, J9.2, TP7.1
- net +5V: now also C51.1, D9.1 (K), J11.2, J12.2, TP6.1, U9.4 (VOUT)
- net GND: now also C1.2, C42.2, C43.2, C44.2, C45.2, C46.2, C47.2, C48.2, C49.2, C50.2, C51.2, J1.10 (SHIELD), J1.4 (GND), J1.7 (DRAIN), J10.1, J11.5, J12.5, J2.4 (GND), J2.5 (Shield), J3.4 (GND), J3.5 (Shield), J4.10 (SHIELD), J4.4 (GND), J4.7 (DRAIN), J5.10 (SHIELD), J5.4 (GND), J5.7 (DRAIN), J6.4 (GND), J6.5 (Shield), J7.10 (SHIELD), J7.4 (GND), J7.7 (DRAIN), J8.10 (SHIELD), J8.4 (GND), J8.7 (DRAIN), J9.1, R42.1, R43.1, R44.1, R45.2, R46.1, R47.2, U9.3 (GND)
- net PWR_1: now also C44.1, J4.1 (VBUS)
- net PWR_2: now also C47.1, J7.1 (VBUS)
- net PWR_3: now also C45.1, J5.1 (VBUS)
- net PWR_4: now also C48.1, J8.1 (VBUS)
- net PWR_5: now also C42.1, J2.1 (VBUS)
- net PWR_6: now also C46.1, J6.1 (VBUS)
- net PWR_7: now also C43.1, J3.1 (VBUS)
- net USB2DM_N1: now also J4.2 (D-)
- net USB2DM_N2: now also J7.2 (D-)
- net USB2DM_N3: now also J5.2 (D-)
- net USB2DM_N4: now also J8.2 (D-)
- net USB2DM_N5: now also J2.2 (D-)
- net USB2DM_N6: now also J6.2 (D-)
- net USB2DM_N7: now also J3.2 (D-)
- net USB2DM_UP: now also J1.3 (D+)
- net USB2DP_N1: now also J4.3 (D+)
- net USB2DP_N2: now also J7.3 (D+)
- net USB2DP_N3: now also J5.3 (D+)
- net USB2DP_N4: now also J8.3 (D+)
- net USB2DP_N5: now also J2.3 (D+)
- net USB2DP_N6: now also J6.3 (D+)
- net USB2DP_N7: now also J3.3 (D+)
- net USB2DP_UP: now also J1.2 (D-)
- net USB3DM_RXN1: now also J4.5 (SSRX-)
- net USB3DM_RXN2: now also J7.5 (SSRX-)
- net USB3DM_RXN3: now also J5.5 (SSRX-)
- net USB3DM_RXN4: now also J8.5 (SSRX-)
- net USB3DM_RXUP: now also U1.67 (USB3DM_RXUP), J1.5 (SSRX-)
- net USB3DM_TXN1: now also J4.8 (SSTX-)
- net USB3DM_TXN2: now also J7.8 (SSTX-)
- net USB3DM_TXN3: now also J5.8 (SSTX-)
- net USB3DM_TXN4: now also J8.8 (SSTX-)
- net USB3DM_TXUP: now also C14.1, J1.8 (SSTX-); no longer U1.64 (USB3DM_TXUP)
- net USB3DP_RXN1: now also J4.6 (SSRX+)
- net USB3DP_RXN2: now also J7.6 (SSRX+)
- net USB3DP_RXN3: now also J5.6 (SSRX+)
- net USB3DP_RXN4: now also J8.6 (SSRX+)
- net USB3DP_RXUP: now also U1.66 (USB3DP_RXUP), J1.6 (SSRX+)
- net USB3DP_TXN1: now also J4.9 (SSTX+)
- net USB3DP_TXN2: now also J7.9 (SSTX+)
- net USB3DP_TXN3: now also J5.9 (SSTX+)
- net USB3DP_TXN4: now also J8.9 (SSTX+)
- net USB3DP_TXUP: now also C19.1, J1.9 (SSTX+); no longer U1.63 (USB3DP_TXUP)
- net VBUS_UP: now also C1.1, J1.1 (VBUS)
- new net: R42.2, U9.5 (Trim)
- new net: C49.1, C50.1, D8.1 (K), U9.1 (EN), U9.2 (VIN)
- new net: C14.2, U1.64 (USB3DM_TXUP)
- new net: C19.2, U1.63 (USB3DP_TXUP)
- new net: D11.2 (A), R46.2, R47.1
- new net: D9.2 (A), R43.2
- new net: D10.2 (A), R44.2, R45.1
- new net +BATT: D10.1 (K), D8.2 (A), J10.3, J11.1, J12.1, J9.3
Other:
- removed sheet connectors
- note added: "1.25V"
- note added: "3.3V"
- note added: "5V"
- note added: "MPM3610 breakout based"
- note added: "MPM3610 is an adjustable buck regulator. R2 is determined by R1/ ((Vout/0.798) - 1); using 191o as R1, R2 = 330 for 1.259Vout - USB5537 has range of 1.22 - 1.31, so this is fine - Adafruit board uses 0402 components"
- note added: "Power"
- note added: "Power Status LEDs"
- note added: "THT"
- note added: "Trim R must be 1/10W precision metal film type Input and output caps must be ceramic (murata GRM32) @ > 24V All components should be as close as possible to device"
- note added: "Will require an adapter board to convert from vertical to horizontal mounting"
- note removed: "Ethernet switch is on the Gigablox nano ethernet switch breakout; connects over a simple genderless samtec connector"
- note removed: "I2C port is currently useless, but it's worth breaking out anyway"
- moved on the sheet: C10, C11, C12, C13, C15, C16, C17, C18, C2, C20, C21, C22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

Commit message: most recent updates
Parts:
- added J13: header_01x02, 5_Connectors_misc:AMASS_XT60-F_1x02_P7.20mm_Vertical, symbol 5.connector.interconnect:header_01x02
- added U10, U11, U12, U13: Mounting-holes, 0_misc:plated_hole_3.0x3.6mm, symbol 5.connector.interconnect:Mounting-holes
- C1, C13, C18, C28, C29, C49, C50, C51: footprint 2_Passives_Capacitors_SMD_IPC:C_2012_805_B -> 2_Passives_Capacitors_SMD_IPC:C_2012_805_A
- C10, C12, C14, C17, C19, C2, C20, C21, C22, C24, C26, C3, C30, C31, C32, C33, C34, C35, C36, C37, C38, C39, C4, C40, C41, C5, C7, C8, C9: footprint 2_Passives_Capacitors_SMD_IPC:C_2012_805_B -> 2_Passives_Capacitors_SMD_IPC:C_1005_402_A
- C11, C15, C16, C6: footprint 2_Passives_Capacitors_SMD_IPC:C_1608_603_B -> 2_Passives_Capacitors_SMD_IPC:C_1608_603_A
- J11, J12: footprint 5_Connectors_misc:header_01x04_pitch2.54_tht -> 5_Connectors_misc:header_01x05_pitch2.54_tht
- R1, R10, R11, R12, R13, R14, R15, R16, R17, R18, R19, R2, R20, R21, R22, R23, R24, R25, R26, R27, R28, R29, R3, R30, R31, R32, R33, R34, R35, R36, R37, R38, R39, R4, R40, R41, R5, R6, R7, R8, R9: footprint 2_Passives_Resistors_SMD_IPC:R_1608_603_B -> 2_Passives_Resistors_SMD_IPC:R_1608_603_A
- R43, R46, R47: footprint 2_Passives_Resistors_SMD_IPC:R_2012_805_B -> 2_Passives_Resistors_SMD_IPC:R_2012_805_A
- R44, R45: footprint 2_Passives_Resistors_SMD_IPC:R_6332_2512_B -> 2_Passives_Resistors_SMD_IPC:R_6332_2512_A
- TP1, TP2, TP3, TP4, TP5, TP6, TP7, TP8: footprint 5_Connectors_misc:2mm_smd_pad -> 0_misc:test_point_2mm_square
- Y1: footprint (none) -> project_footprints:OSC_XRCGB25M000F3M00R0
Connections:
- net +BATT: now also J13.2
- net GND: now also J13.1; no longer U2.9 (EP), U3.9 (EP), U4.9 (EP), U5.9 (EP), U6.9 (EP), U7.9 (EP), U8.9 (EP)
- net +3.3V renamed +1.25V
- net USB2DM_N1 renamed USB2_N1_D-
- net USB2DM_N2 renamed USB2_N2_D-
- net USB2DM_N3 renamed USB2_N3_D-
- net USB2DM_N4 renamed USB2_N4_D-
- net USB2DM_N5 renamed USB2_N5_D-
- net USB2DM_N6 renamed USB2_N6_D-
- net USB2DM_N7 renamed USB2_N7_D-
- net USB2DM_UP renamed USB2_UP_D-
- net USB2DP_N1 renamed USB2_N1_D+
- net USB2DP_N2 renamed USB2_N2_D+
- net USB2DP_N3 renamed USB2_N3_D+
- net USB2DP_N4 renamed USB2_N4_D+
- net USB2DP_N5 renamed USB2_N5_D+
- net USB2DP_N6 renamed USB2_N6_D+
- net USB2DP_N7 renamed USB2_N7_D+
- net USB2DP_UP renamed USB2_UP_D+
- net USB3DM_RXN1 renamed USB3_RXN1_D-
- net USB3DM_RXN2 renamed USB3_RXN2
- net USB3_RXN2: no longer U1.17 (USB3DM_RXDN2)
- net USB3DM_RXN3 renamed USB3_RXN3_D-
- net USB3DM_RXN4 renamed USB3_RXN4_D-
- net USB3DM_RXUP renamed USB3_RXUP_D-
- net USB3DM_TXN1 renamed USB3_TXN1_D-
- net USB3DM_TXN2 renamed USB3_TXN2_D-
- net USB3DM_TXN3 renamed USB3_TXN3_D-
- net USB3DM_TXN4 renamed USB3_TXN4_D-
- net USB3DM_TXUP renamed USB3_TXUP_D-
- net USB3DP_RXN1 renamed USB3_RXN1_D+
- net USB3DP_RXN2 renamed USB3_RXN2_D+
- net USB3DP_RXN3 renamed USB3_RXN3_D+
- net USB3DP_RXN4 renamed USB3_RXN4_D+
- net USB3DP_RXUP renamed USB3_RXUP_D+
- net USB3DP_TXN1 renamed USB3_TXN1_D+
- net USB3DP_TXN2 renamed USB3_TXN2_D+
- net USB3DP_TXN3 renamed USB3_TXN3_D+
- net USB3DP_TXN4 renamed USB3_TXN4_D+
- net USB3DP_TXUP renamed USB3_TXUP_D+
- new net USB3_RXN2_D-: U1.17 (USB3DM_RXDN2)
Other:
- note added: "FIND POWER INPUT CONNECTOR LATER"
